Commit message: fix: CMakeLists.txt file
fix control_node = Node()

File: description/ros2_control/robot.ros2_control.xacro (robot description, xacro)
@@ -12,5 +12,5 @@
                 <state_interface name="velocity"/>
             </joint>
-            <joint name="${prefx}right_wheel_joint">
+            <joint name="${prefix}right_wheel_joint">
                 <command_interface name="velocity"/>
                 <state_interface name="position"/>
