Commit message: fix: fix bag

File: install/lucia_controller/share/lucia_controller/ros2_control/robot.ros2_control.xacro (robot description, xacro)
@@ -1,31 +1 @@
-<?xml version="1.0"?>
-<robot xmlns:xacro="http://www.ros.org/wiki/xacro">
-    <xacro:macro name="robot_ros2_control" params="name prefix">
-        <ros2_control name="${name}" type="system">
-            <hardware>
-                <plugin>lucia_controller/RobotController/Hardware</plugin>
-                <!--<param name="serial_port">/dev/ttyUSB0</param>-->
-            </hardware>
-            <joint name="${prefix}left_wheel_joint">
-                <command_interface name="velocity"/>
-                <state_interface name="position"/>
-                <state_interface name="velocity"/>
-            </joint>
-            <joint name="${prefx}right_wheel_joint">
-                <command_interface name="velocity"/>
-                <state_interface name="position"/>
-                <state_interface name="velocity"/>
-            </joint>
-            <sensor name="${prefix}LiDAR">
-                <state_interface name="orientation.x"/>
-                <state_interface name="orientation.y"/>
-                <state_interface name="orientation.z"/>
-                <state_interface name="orientation.w"/>
-                <state_interface name="angular_velocity.x"/>
-                <state_interface name="angular_gelocity.y"/>
-                <state_interface name="angular_velocity.z"/>
-                <param name="frame_id">LiDAR_link</param>
-            </sensor>
-        </ros2_control>
-    </xacro:macro>
-</robot>
+/home/peach/ros2_ws/src/lucia_controller/description/ros2_control/robot.ros2_control.xacro

File: install/lucia_controller/share/lucia_controller/urdf/robot.urdf.xacro (robot description, xacro)
@@ -1,8 +1 @@
-<?xml version="1.0"?>
-<robot xmlns:xacro="http://www.ros.org/wiki/xacro" name="robot">
-    <xacro:arg name="prefix" default="" />
-    <xacro:include filename="$(find lucia_controller)/urdf/robot_description.urdf.xacro" />
-    <xacro:include filename="$(find lucia_controller)/ros2_control/robot.ros2_control.xacro" />
-    <xacro:robot prefix="$(arg prefix)" />
-    <xacro:robot_ros2_control name="Robot" prefix="$(arg prefix)" />
-</robot>
+/home/peach/ros2_ws/src/lucia_controller/description/urdf/robot.urdf.xacro

File: install/lucia_controller/share/lucia_controller/urdf/robot_description.urdf.xacro (robot description, xacro)
@@ -1,132 +1 @@
-<?xml version="1.0"?>
-<robot xmlns:xacro="http://www.ros.org/wiki/xacro">
-    <xacro:macro name="robot" params="prefix">
-        <!-- Constants for robot dimensions -->
-        <xacro:property name="PI" value="3.1415926535897931" />
-        <material name="black">
-            <color rgba="0.0 0.0 0.0 1.0"/>
-        </material>
-        <material name="blue">
-            <color rgba="0.0 0.0 0.8 0.8"/>
-        </material>
-        <material name="brown">
-            <color rgba="${165/255} ${42/255} ${42/255} 1.0"/>
-        </material>
-        <link name="${prefix}base_footprint" />
-        <joint name="${prefix}base_joint" type="fixed">
-            <parent link="${prefix}base_footprint"/>
-            <child link="${prefix}base_link"/>
-            <origin xyz="0 0 0.032" rpy="0 0 0"/>
-        </joint>
-        <!-- Base Link -->
-        <link name="${prefix}base_link">
-            <visual>
-                <origin xyz="-0.07 0 0.038" rpy="0 0 0" />
-                <geometry>
-                    <box size="0.225 0.225 0.125"/>
-                </geometry>
-                <material name="blue"/>
-            </visual>
-            <collision>
-                <origin xyz="-0.07 0 0.038" rpy="0 0 0" />
-                <geometry>
-                    <box size="0.225 0.225 0.125"/>
-                </geometry>
-            </collision>
-        </link>
-        <!-- left wheel Link -->
-        <joint name="${prefix}left_wheel_joint" type="continuous">
-            <parent link="${prefix}base_link"/>
-            <child link="${prefix}left_wheel"/>
-            <origin xyz="0 0.105 0" rpy="0 0 0"/>
-            <axis xyz="0 1 0"/>
-            <dynamics damping="0.2"/>
-        </joint>
-        <link name="${prefix}left_wheel">
-            <collision>
-                <origin xyz="0 0 0" rpy="${pi/2} 0 0"/>
-                <geometry>
-                    <cylinder length="0.01" radius="0.032"/>
-                </geometry>
-            </collision>
-            <visual>
-                <origin xyz="0 0 0" rpy="${pi/2} 0 0"/>
-                <geometry>
-                    <cylinder length="0.01" radius="0.032"/>
-                </geometry>
-                <material name="black"/>
-            </visual>
-        </link>
-        <!-- right wheel Link -->
-        <joint name="${prefix}right_wheel_joint" type="continuous">
-            <parent link="${prefix}base_link"/>
-            <child link="${prefix}right_wheel"/>
-            <origin xyz="0 -0.105 0" rpy="0 0 0"/>
-            <axis xyz="0 1 0"/>
-            <dynamics damping="0.2"/>
-        </joint>
-        <link name="${prefix}right_wheel">
-            <collision>
-                <origin xyz="0 0 0" rpy="${pi/2} 0 0"/>
-                <geometry>
-                    <cylinder length="0.01" radius="0.032"/>
-                </geometry>
-            </collision>
-            <visual>
-                <origin xyz="0 0 0" rpy="${pi/2} 0 0"/>
-                <geometry>
-                    <cylinder length="0.01" radius="0.032"/>
-                </geometry>
-                <material name="black"/>
-            </visual>
-        </link>
-        <joint name="${prefix}right_free_wheel_joint" type="fixed">
-            <parent link="${prefix}base_link"/>
-            <child link="${prefix}right_free_wheel"/>
-            <origin xyz="-0.135 -0.105 -0.02" rpy="0 0 0"/>
-        </joint>
-        <link name="${prefix}right_free_wheel">
-            <visual>
-                <origin xyz="0 0 0" rpy="${pi/2} 0 0"/>
-                <geometry>
-                    <cylinder length="0.01" radius="0.01"/>
-                </geometry>
-                <material name="brown"/>
-            </visual>
-        </link>
-        <joint name="${prefix}left_free_wheel_joint" type="fixed">
-            <parent link="${prefix}base_link"/>
-            <child link="${prefix}left_free_wheel"/>
-            <origin xyz="-0.135 0.105 -0.02" rpy="0 0 0"/>
-        </joint>
-        <link name="${prefix}left_free_wheel">
-            <visual>
-                <origin xyz="0 0 0" rpy="${pi/2} 0 0"/>
-                <geometry>
-                    <cylinder length="0.01" radius="0.01"/>
-                </geometry>
-                <material name="brown"/>
-            </visual>
-        </link>
-        <link name="${prefix}imu_link" />
-        <joint name="${prefix}imu_joint" type="fixed">
-            <parent link="${prefix}base_link"/>
-            <child link="${prefix}imu_link"/>
-            <origin xyz="-0.062 -0.064 0.01" rpy="0 0 0"/>
-        </joint>
-        <link name="${prefix}laser_link">
-            <visual>
-                <origin xyz="0 0 -0.02" rpy="0 0 0" />
-                <geometry>
-                    <cylinder length="0.04" radius="0.025"/>
-                </geometry>
-                <material name="black"/>
-            </visual>
-        </link>
-        <joint name="${prefix}laser_joint" type="fixed">
-            <parent link="${prefix}base_link"/>
-            <child link="${prefix}laser_link"/>
-            <origin xyz="-0.135 0 0.14" rpy="0 0 ${PI}"/>
-        </joint>
-    </xacro:macro>
-</robot>
+/home/peach/ros2_ws/src/lucia_controller/description/urdf/robot_description.urdf.xacro
