Commit message: fix

File: description/urdf/lucia.urdf (robot description, URDF)
Before this commit: robot lucia, 5 links, 4 joints
Links:
- removed link body_link
- removed link lidar
- added link base_footprint; visual cylinder length=1.0 radius=0.5
- added link laser; visual cylinder length=0.1 radius=0.1
Joints:
- joint body_joint: child body_link -> base_footprint
- joint lidar_joint: child lidar -> laser
